File: RicardoTemplate.kicad_sch (KiCad schematic)
At the start: 38 parts, among them J1 RBUS, U1 ESP32-S3, U5 LTC4411, Y1 40MHz±10ppm

Commit message: tidied up
Parts:
- added C?: 1uF, Capacitor_SMD:C_0603_1608Metric, symbol Device:C_Small
- added C?: 10uF, Capacitor_SMD:C_0603_1608Metric, symbol Device:C_Small
- added C?: 10nF, Capacitor_SMD:C_0603_1608Metric, symbol Device:C_Small
- added C?: 0.1uF, Capacitor_SMD:C_0603_1608Metric, symbol Device:C_Small
- added C?: 2.2uF, Capacitor_SMD:C_0603_1608Metric, symbol Device:C_Small
- added C?: 0.47uF, Capacitor_SMD:C_0603_1608Metric, symbol Device:C_Small
- added J?: Micro_SD_Card_Det, Connector_Card:microSD_HC_Hirose_DM3AT-SF-PEJM5, symbol Connector:Micro_SD_Card_Det_Hirose_DM3AT
- added R?: 10k, symbol Device:R_Small
- added U?: ICM-20608-G, iclr:PQFN50P300X300X80-16N, symbol iclr:ICM-20608-G
- added U?: MMC5983MA, iclr:PQFN50P300X300X100-16N, symbol iclr:MMC5983MA
Connections:
- net +3V3: now also C?.1, C?.1, C?.1, C?.1, J?.4 (VDD), R?.1, U?.1 (VDDIO), U?.13 (VDDIO), U?.16 (VDD), U?.2 (VDD)
- net GND: now also C?.2, C?.2, J?.11 (SHIELD), J?.6 (VSS), J?.9 (DET_B), U?.10 (GND), U?.11 (GND), U?.11 (GND), U?.12 (GND), U?.13 (GND), U?.15 (GND), U?.8 (FSYNC), U?.9 (GND), U?.9 (GND)
- net SPI_CLK: now reaches U1.38 (GPIO33)
- net SPI_CLK: now also J?.5 (CLK), U?.1 (SCL/SPI_SCK), U?.2 (SCL/SCLK)
- net SPI_MOSI: now reaches U1.39 (GPIO34)
- net SPI_MOSI: now also J?.3 (CMD), U?.16 (SDA/SPI_SDI), U?.3 (SDA/SDI)
- net SPI_MISO: now reaches U1.40 (GPIO35)
- net SPI_MISO: now also J?.7 (DAT0), U?.4 (AD0/SDO), U?.5 (SPI_SDO)
- net IMU_CS: now reaches U1.41 (GPIO36)
- net IMU_CS: now also U?.5 (CS)
- net MAG_CS: now reaches U1.42 (GPIO37)
- net MAG_CS: now also U?.4 (~{SPI_CS})
- net SD_CS: now reaches U1.43 (GPIO38)
- net SD_CS: now also J?.2 (DAT3/CD)
- new net: C?.1, U?.14 (REGOUT)
- new net: C?.1, U?.10 (CAP)
- new net: C?.2, C?.2, C?.2, C?.2
- new net: J?.10 (DET_A), R?.2
- new net: U?.12 (NC), U?.14 (NC), U?.3 (NC), U?.6 (NC), U?.7 (NC), U?.8 (NC)
- no-connect marks 4 -> 8
