File: _autosave-Canardboard.kicad_sch (KiCad schematic)
At the start: 58 parts, among them J1 RBUS, J4 Conn_01x02_Male, J5 Conn_01x03_Male, J6 Conn_01x03_Male, J7 Conn_01x03_Male, Q1 SI4143DY-T1-GE3, Q2 SI4143DY-T1-GE3, U1 ESP32-S3, U10 LTC4412xS6, U9 LTC4412xS6, Y1 40MHz±10ppm

Commit message: first draft of PCB layout
Parts:
- J1: footprint Connector_Molex:Molex_Mini-Fit_Jr_5566-06A_2x03_P4.20mm_Vertical -> Connector_Molex:Molex_Mini-Fit_Jr_5569-06A2_2x03_P4.20mm_Horizontal
Connections:
- net RBUS_PWR is gone; now on net RBUS_DEPL: Q1.1 (S), Q1.2 (S), Q1.3 (S), U9.1 (VIN)
- net +12V: no longer J1.4 (Pin_4)
- net RBUS_DEPL: now also J1.4 (Pin_4)
- no-connect marks 31 -> 32
Other:
- moved on the sheet: Y1
Changed lines of the file:
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@@
   )
   (no_connect (at 135.89 80.01))
+  (no_connect (at 69.85 115.57))
   (no_connect (at 135.89 77.47))
   (no_connect (at 135.89 87.63))
@@
     (effects (font (size 1.27 1.27)) (justify right bottom))
   )
+  (label "RBUS_DEPL" (at 242.57 36.83 180) (fields_autoplaced)
+    (effects (font (size 1.27 1.27)) (justify right bottom))
+  )
   (label "SERVO_SGNL2" (at 259.08 142.24 180) (fields_autoplaced)
     (effects (font (size 1.27 1.27)) (justify right bottom))
@@
     (effects (font (size 1.27 1.27)) (justify left bottom))
   )
-  (label "RBUS_DEPL" (at 120.65 27.94 270) (fields_autoplaced)
+  (label "RBUS_DEPL" (at 120.65 25.4 270) (fields_autoplaced)
     (effects (font (size 1.27 1.27)) (justify right bottom))
   )
@@
     )
   )
-  (hierarchical_label "RBUS_PWR" (shape input) (at 242.57 36.83 180) (fields_autoplaced)
-    (effects (font (size 1.27 1.27)) (justify right))
-  )
   (symbol (lib_id "power:+3.3V") (at 30.48 182.88 0) (unit 1)
     (in_bom yes) (on_board yes) (dnp no)
@@
       (effects (font (size 1.27 1.27)))
     )
-    (property "Footprint" "Connector_Molex:Molex_Mini-Fit_Jr_5566-06A_2x03_P4.20mm_Vertical" (at 123.19 20.32 0)
+    (property "Footprint" "Connector_Molex:Molex_Mini-Fit_Jr_5569-06A2_2x03_P4.20mm_Horizontal" (at 123.19 20.32 0)
       (effects (font (size 1.27 1.27)) hide)
     )
@@
         (path "/7db990e4-92e1-4f99-b4d2-435bbec1ba83"
           (reference "#PWR078") (unit 1)
-        )
-      )
-    )
-  )
-  (symbol (lib_id "power:+12V") (at 120.65 25.4 180) (unit 1)
-    (in_bom yes) (on_board yes) (dnp no)
-    (property "Reference" "#PWR017" (at 120.65 21.59 0)
-      (effects (font (size 1.27 1.27)) hide)
-    )
-    (property "Value" "+12V" (at 120.65 31.75 90)
-      (effects (font (size 1.27 1.27)) hide)
-    )
-    (property "Footprint" "" (at 120.65 25.4 0)
-      (effects (font (size 1.27 1.27)) hide)
-    )
-    (property "Datasheet" "" (at 120.65 25.4 0)
-      (effects (font (size 1.27 1.27)) hide)
-    )
-    (pin "1")
-    (instances
-      (project "Canardboard"
-        (path "/7db990e4-92e1-4f99-b4d2-435bbec1ba83"
-          (reference "#PWR017") (unit 1)
         )
       )
@@
     )
   )
-  (symbol (lib_id "Device:Crystal_GND24") (at 156.21 132.08 90) (unit 1)
-    (in_bom yes) (on_board yes) (dnp no)
-    (property "Reference" "Y1" (at 152.4 121.92 90)
-      (effects (font (size 1.27 1.27)))
-    )
-    (property "Value" "40MHz±10ppm" (at 152.4 124.46 90)
-      (effects (font (size 1.27 1.27)))
-    )
+  (symbol (lib_id "Device:Crystal_GND24") (at 156.21 132.08 270) (mirror x) (unit 1)
+    (in_bom yes) (on_board yes) (dnp no)
+    (property "Reference" "Y1" (at 160.02 121.92 90)
+      (effects (font (size 1.27 1.27)))
+    )
+    (property "Value" "40MHz±10ppm" (at 160.02 124.46 90)
+      (effects (font (size 1.27 1.27)))
+    )
