File: power.kicad_sch (KiCad schematic)
At the start: 21 parts, among them U3 LM66200DRLR, U5 MAX77827AEFD+T, U6 SC4215

Commit message: error encountered - battery logic and inductor
- use large capacitor?
- use VBUS as a power source?
Parts:
- removed C20, C25, C27: 10uF, Capacitor_SMD:C_0402_1005Metric, symbol Device:C_Small
- removed C22: 10uF, Capacitor_SMD:C_0603_1608Metric, symbol Device:C_Small
- removed C23: 1uF, Capacitor_SMD:C_0402_1005Metric, symbol Device:C_Small
- removed C24: 22uF, Capacitor_SMD:C_0603_1608Metric, symbol Device:C_Small
- removed C26: 4.7uF, Capacitor_SMD:C_0402_1005Metric, symbol Device:C_Small
- removed C28: 0.1uF, Capacitor_SMD:C_0402_1005Metric, symbol Device:C_Small
- removed L3: 1uH, Inductor_SMD:L_0805_2012Metric, symbol Device:L
- removed R14: 14k, Resistor_SMD:R_0402_1005Metric, symbol Device:R_Small
- removed R15: 56k, Resistor_SMD:R_0402_1005Metric, symbol Device:R_Small
- removed R16, R23: 10k, Resistor_SMD:R_0402_1005Metric, symbol Device:R_Small
- removed TP4, TP5, TP6, TP7, TP8: TestPoint, TestPoint:TestPoint_Pad_D1.5mm, symbol Connector:TestPoint
- removed U3: LM66200DRLR, iclr:SOTFL50P160X60-8N, symbol iclr:LM66200DRLR
- removed U5: MAX77827AEFD+T, iclr:CONV_MAX77827AEFD+T, symbol iclr:MAX77827AEFD+T
- removed U6: SC4215, iclr:SOIC127P599X175-9N, symbol iclr:RT9025-25GSP
Connections:
- no-connect marks 4 -> 0
Other:
- note removed: "Be extra careful in leaving this connected at a single point"
