File: servopower.kicad_sch (KiCad schematic)
At the start: 45 parts, among them IC1 SIC437DED-T1-GE3, U10 MP28167GQ-A-Z

Commit message: I don't want to lose all my changes so I will commit, commit.
Parts:
- removed C47: 100uF, Capacitor_SMD:CP_Elec_6.3x5.4, symbol Device:C_Small
- added C42 (x2): 47uF, Capacitor_SMD:C_1206_3216Metric, symbol Device:C_Small
- L4: footprint iclr:INDPM112100X400N -> iclr:INDPM3030X200N
Connections:
- net GND: now also C42.2, C42.2
- net RBUS_uC_V: now also C42.1, C42.1
Changed lines of the file:
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@@
   (junction (at 186.69 111.76) (diameter 0) (color 0 0 0 0)
   )
+  (junction (at 123.19 31.75) (diameter 0) (color 0 0 0 0)
+  )
   (junction (at 149.86 125.73) (diameter 0) (color 0 0 0 0)
   )
@@
   )
   (junction (at 173.99 147.32) (diameter 0) (color 0 0 0 0)
+  )
+  (junction (at 123.19 36.83) (diameter 0) (color 0 0 0 0)
   )
   (junction (at 156.21 31.75) (diameter 0) (color 0 0 0 0)
@@
     (stroke (width 0) (type default))
   )
+  (wire (pts (xy 123.19 31.75) (xy 133.35 31.75))
+    (stroke (width 0) (type default))
+  )
   (wire (pts (xy 133.35 36.83) (xy 143.51 36.83))
     (stroke (width 0) (type default))
@@
     (stroke (width 0) (type default))
   )
-  (wire (pts (xy 123.19 31.75) (xy 133.35 31.75))
-    (stroke (width 0) (type default))
-  )
   (wire (pts (xy 149.86 128.27) (xy 149.86 132.08))
     (stroke (width 0) (type default))
@@
     (stroke (width 0) (type default))
   )
+  (wire (pts (xy 113.03 36.83) (xy 123.19 36.83))
+    (stroke (width 0) (type default))
+  )
   (wire (pts (xy 149.86 123.19) (xy 154.94 123.19))
     (stroke (width 0) (type default))
   )
   (wire (pts (xy 170.18 132.08) (xy 191.77 132.08))
+    (stroke (width 0) (type default))
+  )
+  (wire (pts (xy 113.03 31.75) (xy 123.19 31.75))
     (stroke (width 0) (type default))
   )
@@
     (effects (font (size 1.27 1.27)) (justify right bottom))
   )
-  (global_label "RBUS_uC_V" (shape input) (at 123.19 31.75 180) (fields_autoplaced)
+  (global_label "RBUS_uC_V" (shape input) (at 113.03 31.75 180) (fields_autoplaced)
     (effects (font (size 1.27 1.27)) (justify right))
-    (property "Intersheetrefs" "${INTERSHEET_REFS}" (at 110.4156 31.75 0)
+    (property "Intersheetrefs" "${INTERSHEET_REFS}" (at 100.2556 31.75 0)
       (effects (font (size 1.27 1.27)) (justify right) hide)
     )
@@
         (path "/7db990e4-92e1-4f99-b4d2-435bbec1ba83/9ac1c7a8-1287-4655-8906-f7f2eef1324f"
           (reference "R33") (unit 1)
+        )
+      )
+    )
+  )
+  (symbol (lib_id "Device:C_Small") (at 113.03 34.29 0) (unit 1)
+    (in_bom yes) (on_board yes) (dnp no) (fields_autoplaced)
+    (property "Reference" "C42" (at 115.57 33.6613 0)
+      (effects (font (size 1.27 1.27)) (justify left))
+    )
+    (property "Value" "47uF" (at 115.57 36.2013 0)
+      (effects (font (size 1.27 1.27)) (justify left))
+    )
+    (property "Footprint" "Capacitor_SMD:C_1206_3216Metric" (at 113.03 34.29 0)
+      (effects (font (size 1.27 1.27)) hide)
+    )
+    (property "Datasheet" "~" (at 113.03 34.29 0)
+      (effects (font (size 1.27 1.27)) hide)
+    )
+    (pin "1")
+    (pin "2")
+    (instances
+      (project "Canardboard"
+        (path "/7db990e4-92e1-4f99-b4d2-435bbec1ba83/e0402675-af14-46ad-ab53-2a6080ba54c9"
+          (reference "C42") (unit 1)
+        )
+        (path "/7db990e4-92e1-4f99-b4d2-435bbec1ba83/9ac1c7a8-1287-4655-8906-f7f2eef1324f"
+          (reference "C19") (unit 1)
         )
       )
@@
     )
   )
-  (symbol (lib_id "Device:C_Small") (at 123.19 34.29 0) (unit 1)
-    (in_bom yes) (on_board yes) (dnp no) (fields_autoplaced)
-    (property "Reference" "C47" (at 125.73 33.6613 0)
-      (effects (font (size 1.27 1.27)) (justify left))
-    )
-    (property "Value" "100uF" (at 125.73 36.2013 0)
-      (effects (font (size 1.27 1.27)) (justify left))
-    )
-    (property "Footprint" "Capacitor_SMD:CP_Elec_6.3x5.4" (at 123.19 34.29 0)
-      (effects (font (size 1.27 1.27)) hide)
-    )
-    (property "Datasheet" "~" (at 123.19 34.29 0)
-      (effects (font (size 1.27 1.27)) hide)
-    )
-    (pin "1")
-    (pin "2")
-    (instances
-      (project "Canardboard"
-        (path "/7db990e4-92e1-4f99-b4d2-435bbec1ba83/9ac1c7a8-1287-4655-8906-f7f2eef1324f"
-          (reference "C47") (unit 1)
-        )
-      )
-    )
-  )
   (symbol (lib_name "GND_1") (lib_id "power:GND") (at 147.32 161.29 0) (unit 1)
     (in_bom yes) (on_board yes) (dnp no) (fields_autoplaced)
@@
     )
   )
+  (symbol (lib_id "Device:C_Small") (at 123.19 34.29 0) (unit 1)
+    (in_bom yes) (on_board yes) (dnp no) (fields_autoplaced)
+    (property "Reference" "C42" (at 125.73 33.6613 0)
+      (effects (font (size 1.27 1.27)) (justify left))
+    )
+    (property "Value" "47uF" (at 125.73 36.2013 0)
+      (effects (font (size 1.27 1.27)) (justify left))
+    )
+    (property "Footprint" "Capacitor_SMD:C_1206_3216Metric" (at 123.19 34.29 0)
+      (effects (font (size 1.27 1.27)) hide)
+    )
+    (property "Datasheet" "~" (at 123.19 34.29 0)
+      (effects (font (size 1.27 1.27)) hide)
+    )
+    (pin "1")
+    (pin "2")
+    (instances
+      (project "Canardboard"
+        (path "/7db990e4-92e1-4f99-b4d2-435bbec1ba83/e0402675-af14-46ad-ab53-2a6080ba54c9"
+          (reference "C42") (unit 1)
+        )
+        (path "/7db990e4-92e1-4f99-b4d2-435bbec1ba83/9ac1c7a8-1287-4655-8906-f7f2eef1324f"
+          (reference "C18") (unit 1)
+        )
+      )
+    )
+  )
   (symbol (lib_id "Device:R_Small") (at 167.64 53.34 90) (unit 1)
     (in_bom yes) (on_board yes) (dnp no) (fields_autoplaced)
@@
       (effects (font (size 1.27 1.27)))
     )
-    (property "Footprint" "iclr:INDPM112100X400N" (at 195.58 132.08 0)
-      (effects (font (size 1.27 1.27)) hide)
-    )
+    (property "Footprint" "iclr:INDPM3030X200N" (at 195.58 132.08 0)
+      (effects (font (size 1.27 1.27)) hide)
+    )

Commit message: i dont know
Parts:
- L4: footprint iclr:INDPM3030X200N -> iclr:INDPM112100X400N
Changed lines of the file:
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@@
       (effects (font (size 1.27 1.27)))
     )
-    (property "Footprint" "iclr:INDPM3030X200N" (at 195.58 132.08 0)
+    (property "Footprint" "iclr:INDPM112100X400N" (at 195.58 132.08 0)
       (effects (font (size 1.27 1.27)) hide)
     )

Commit message: weird 3v3 and 3.3v bug
Other:
- moved on the sheet: C42, C43
