File: _autosave-servopower.kicad_sch (KiCad schematic)
At the start: 53 parts, among them IC1 SIC437DED-T1-GE3, U10 MP28167GQ-A-Z, U9 SC4215

Commit message: fixed all of andrei's comments v1
Parts:
- removed TP16: TestPoint, TestPoint:TestPoint_Pad_D2.0mm, symbol Connector:TestPoint
- added JP1: TermJP, Jumper:SolderJumper-2_P1.3mm_Open_RoundedPad1.0x1.5mm, symbol Jumper:SolderJumper_2_Open
Connections:
- net +3V3: now also JP1.2 (B)
- net uC_VOUT: now also JP1.1 (A)
Changed lines of the file:
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@@
   (junction (at 205.74 147.32) (diameter 0) (color 0 0 0 0)
-  )
-  (junction (at 274.32 50.8) (diameter 0) (color 0 0 0 0)
   )
   (junction (at 149.86 128.27) (diameter 0) (color 0 0 0 0)
@@
     )
   )
+  (symbol (lib_id "power:+3.3V") (at 191.77 43.18 0) (unit 1)
+    (in_bom yes) (on_board yes) (dnp no) (fields_autoplaced)
+    (property "Reference" "#PWR096" (at 191.77 46.99 0)
+      (effects (font (size 1.27 1.27)) hide)
+    )
+    (property "Value" "+3.3V" (at 191.77 39.6042 0)
+      (effects (font (size 1.27 1.27)))
+    )
+    (property "Footprint" "" (at 191.77 43.18 0)
+      (effects (font (size 1.27 1.27)) hide)
+    )
+    (property "Datasheet" "" (at 191.77 43.18 0)
+      (effects (font (size 1.27 1.27)) hide)
+    )
+    (pin "1")
+    (instances
+      (project "Canardboard"
+        (path "/7db990e4-92e1-4f99-b4d2-435bbec1ba83/9ac1c7a8-1287-4655-8906-f7f2eef1324f"
+          (reference "#PWR096") (unit 1)
+        )
+      )
+    )
+  )
   (symbol (lib_id "Device:R_Small") (at 248.92 121.92 90) (unit 1)
     (in_bom yes) (on_board yes) (dnp no)
@@
         (path "/7db990e4-92e1-4f99-b4d2-435bbec1ba83/9ac1c7a8-1287-4655-8906-f7f2eef1324f"
           (reference "C56") (unit 1)
+        )
+      )
+    )
+  )
+  (symbol (lib_id "Jumper:SolderJumper_2_Open") (at 191.77 46.99 90) (unit 1)
+    (in_bom yes) (on_board yes) (dnp no) (fields_autoplaced)
+    (property "Reference" "JP1" (at 194.31 46.355 90)
+      (effects (font (size 1.27 1.27)) (justify right))
+    )
+    (property "Value" "TermJP" (at 194.31 48.895 90)
+      (effects (font (size 1.27 1.27)) (justify right))
+    )
+    (property "Footprint" "Jumper:SolderJumper-2_P1.3mm_Open_RoundedPad1.0x1.5mm" (at 191.77 46.99 0)
+      (effects (font (size 1.27 1.27)) hide)
+    )
+    (property "Datasheet" "~" (at 191.77 46.99 0)
+      (effects (font (size 1.27 1.27)) hide)
+    )
+    (pin "1")
+    (pin "2")
+    (instances
+      (project "Canardboard"
+        (path "/7db990e4-92e1-4f99-b4d2-435bbec1ba83/00000000-0000-0000-0000-000061942b9a"
+          (reference "JP1") (unit 1)
+        )
+        (path "/7db990e4-92e1-4f99-b4d2-435bbec1ba83/9ac1c7a8-1287-4655-8906-f7f2eef1324f"
+          (reference "JP2") (unit 1)
         )
       )
@@
         )
       )
-    )
-  )
-  (symbol (lib_id "Connector:TestPoint") (at 274.32 50.8 180) (unit 1)
-    (in_bom yes) (on_board yes) (dnp no)
-    (property "Reference" "TP16" (at 284.48 54.61 0)
-      (effects (font (size 1.27 1.27)) (justify left))
-    )
-    (property "Value" "TestPoint" (at 284.48 52.0731 0)
-      (effects (font (size 1.27 1.27)) (justify left))
-    )
-    (property "Footprint" "TestPoint:TestPoint_Pad_D2.0mm" (at 269.24 50.8 0)
-      (effects (font (size 1.27 1.27)) hide)
-    )
-    (property "Datasheet" "~" (at 269.24 50.8 0)
-      (effects (font (size 1.27 1.27)) hide)
-    )
-    (pin "1")
-    (instances
-      (project "Canardboard"
-        (path "/7db990e4-92e1-4f99-b4d2-435bbec1ba83/9ac1c7a8-1287-4655-8906-f7f2eef1324f"
-          (reference "TP16") (unit 1)
-        )
-      )
-      (project "PickleRick"
-        (path "/e63e39d7-6ac0-4ffd-8aa3-1841a4541b55/150d7a0e-7d8c-4788-bc30-4a3682bf4d09"
-          (reference "TP13") (unit 1)
-        )
-      )
-      (project "power"
-        (path "/e9284afa-e324-4762-b662-a428eebcb5c2"
-          (reference "TP13") (unit 1)
-        )
-      )
