File: can.kicad_sch (KiCad schematic)
At the start: 11 parts, among them U2 SN65HVD230

Commit message: schematic review updated
fixed:
-pin 1 on the bootjumper is missing a connection. 
- Move the SD card to a 2nd SPI bus (so a 2nd set of MISO, MOSI, SCLK) as the rest of the bus is blocked while data is written to it, which would interrupt sensor readings. 
- Add a pull-up resistor on the DET_A pin of the micro SD card, and also connect that pin to the esp32 (picture from pickle) 
- VDD on the IMU (U7) is not connected to any power, should be connected to 3.3V 
- Turns out CAN capacitors C18, C19 actually aren’t needed. It’s up to you if you want to keep them, but if you do keep them could you change their value to “DNP” (stands for Do not place) 
-  Add test points to lines which can potentially cause issues. Most of the time this just means places that are connected to the ESP32, but especially places like the SPI lines (including chip selects). Also, add test points to TXD and RXD on the esp32 in case we have to solder to them for programming  

Servo Buck Converter 
- Pin 29 missing ground connection 
-  Add a text label with the part number of the 2.1uH inductor 

LTC4412s 
- No power net connected to Vin 
- stocky diodes replaced logic mosfets
- switched mosfets around so S is common
Parts:
- removed C18, C19: 220pF, Capacitor_SMD:C_0402_1005Metric, symbol Device:C_Small
Changed lines of the file:
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@@
-    (stroke (width 0) (type default))
-  )
-  (wire (pts (xy 175.26 85.09) (xy 175.26 88.9))
     (stroke (width 0) (type default))
   )
@@
     )
   )
-  (symbol (lib_id "Device:C_Small") (at 175.26 82.55 180) (unit 1)
-    (in_bom yes) (on_board yes) (dnp no)
-    (property "Reference" "C18" (at 173.99 74.93 0)
-      (effects (font (size 1.27 1.27)) (justify right))
-    )
-    (property "Value" "220pF" (at 173.99 77.47 0)
-      (effects (font (size 1.27 1.27)) (justify right))
-    )
-    (property "Footprint" "Capacitor_SMD:C_0402_1005Metric" (at 175.26 82.55 0)
-      (effects (font (size 1.27 1.27)) hide)
-    )
-    (property "Datasheet" "~" (at 175.26 82.55 0)
-      (effects (font (size 1.27 1.27)) hide)
-    )
-    (pin "1")
-    (pin "2")
-    (instances
-      (project "Canardboard"
-        (path "/7db990e4-92e1-4f99-b4d2-435bbec1ba83/00000000-0000-0000-0000-000061942b9a"
-          (reference "C18") (unit 1)
-        )
-      )
-    )
-  )
   (symbol (lib_id "Diode:SM712_SOT23") (at 186.69 88.9 270) (unit 1)
     (in_bom yes) (on_board yes) (dnp no) (fields_autoplaced)
@@
         (path "/7db990e4-92e1-4f99-b4d2-435bbec1ba83/00000000-0000-0000-0000-000061942b9a"
           (reference "#PWR027") (unit 1)
-        )
-      )
-    )
-  )
-  (symbol (lib_id "power:GND") (at 175.26 102.87 0) (unit 1)
-    (in_bom yes) (on_board yes) (dnp no) (fields_autoplaced)
-    (property "Reference" "#PWR028" (at 175.26 109.22 0)
-      (effects (font (size 1.27 1.27)) hide)
-    )
-    (property "Value" "GND" (at 175.26 106.68 0)
-      (effects (font (size 1.27 1.27)))
-    )
-    (property "Footprint" "" (at 175.26 102.87 0)
-      (effects (font (size 1.27 1.27)) hide)
-    )
-    (property "Datasheet" "" (at 175.26 102.87 0)
-      (effects (font (size 1.27 1.27)) hide)
-    )
-    (pin "1")
-    (instances
-      (project "Canardboard"
-        (path "/7db990e4-92e1-4f99-b4d2-435bbec1ba83/00000000-0000-0000-0000-000061942b9a"
-          (reference "#PWR028") (unit 1)
         )
       )
@@
         )
       )
-    )
-  )
-  (symbol (lib_id "Device:C_Small") (at 175.26 100.33 180) (unit 1)
-    (in_bom yes) (on_board yes) (dnp no) (fields_autoplaced)
-    (property "Reference" "C19" (at 177.8 99.0535 0)
-      (effects (font (size 1.27 1.27)) (justify right))
-    )
-    (property "Value" "220pF" (at 177.8 101.5935 0)
-      (effects (font (size 1.27 1.27)) (justify right))
-    )
-    (property "Footprint" "Capacitor_SMD:C_0402_1005Metric" (at 175.26 100.33 0)
-      (effects (font (size 1.27 1.27)) hide)
-    )
-    (property "Datasheet" "~" (at 175.26 100.33 0)
-      (effects (font (size 1.27 1.27)) hide)
-    )
-    (pin "1")
-    (pin "2")
-    (instances
-      (project "Canardboard"
-        (path "/7db990e4-92e1-4f99-b4d2-435bbec1ba83/00000000-0000-0000-0000-000061942b9a"
-          (reference "C19") (unit 1)
-        )
-      )

Commit message: fixed all of andrei's comments v1
Parts:
- R8: footprint Resistor_SMD:R_0603_1608Metric -> Resistor_SMD:R_0402_1005Metric
Changed lines of the file:
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@@
       (effects (font (size 1.27 1.27)) (justify left))
     )
-    (property "Footprint" "Resistor_SMD:R_0603_1608Metric" (at 124.46 95.25 0)
+    (property "Footprint" "Resistor_SMD:R_0402_1005Metric" (at 124.46 95.25 0)
       (effects (font (size 1.27 1.27)) hide)
     )

Commit message: final andrei changes
lol
Parts:
- JP1: footprint Jumper:SolderJumper-2_P1.3mm_Open_RoundedPad1.0x1.5mm -> iclr:SmallerSolderJP
Changed lines of the file:
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@@
       (effects (font (size 1.27 1.27)))
     )
-    (property "Footprint" "Jumper:SolderJumper-2_P1.3mm_Open_RoundedPad1.0x1.5mm" (at 157.48 88.9 0)
+    (property "Footprint" "iclr:SmallerSolderJP" (at 157.48 88.9 0)
       (effects (font (size 1.27 1.27)) hide)
     )
