File: Canardboard.kicad_sch (KiCad schematic)
At the start: 53 parts, among them J5 Conn_01x03_Male, J6 Conn_01x03_Male, J7 Conn_01x03_Male, U1 ESP32-S3, Y1 40MHz±10ppm

Commit message: new board just dropped
i hate my life
Connections:
- net IMU_CS: now also U1.37 (SPICLK_P/GPIO47); no longer U1.38 (GPIO33)
- net MAG_CS: now also U1.36 (SPICLK_N/GPIO48); no longer U1.37 (SPICLK_P/GPIO47)
- net SPI_CLK: now also U1.40 (GPIO35); no longer U1.39 (GPIO34)
- net SPI_MISO: now also U1.38 (GPIO33); no longer U1.36 (SPICLK_N/GPIO48)
- net SPI_MOSI: now also U1.39 (GPIO34); no longer U1.40 (GPIO35)
Changed lines of the file:
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@@
     (effects (font (size 1.27 1.27)) (justify right bottom))
+  )
+  (label "IMU_CS" (at 135.89 118.11 0) (fields_autoplaced)
+    (effects (font (size 1.27 1.27)) (justify left bottom))
   )
   (label "CAN+" (at 115.57 185.42 0) (fields_autoplaced)
@@
     (effects (font (size 1.27 1.27)) (justify left bottom))
   )
+  (label "SPI_MOSI" (at 135.89 97.79 0) (fields_autoplaced)
+    (effects (font (size 1.27 1.27)) (justify left bottom))
+  )
   (label "Data+" (at 99.06 160.02 0) (fields_autoplaced)
     (effects (font (size 1.27 1.27)) (justify left bottom))
@@
   (label "SD_MOSI" (at 227.33 39.37 180) (fields_autoplaced)
     (effects (font (size 1.27 1.27)) (justify right bottom))
+  )
+  (label "SPI_MISO" (at 135.89 95.25 0) (fields_autoplaced)
+    (effects (font (size 1.27 1.27)) (justify left bottom))
   )
   (label "CAN+" (at 227.33 88.9 0) (fields_autoplaced)
@@
     (effects (font (size 1.27 1.27)) (justify right bottom))
   )
-  (label "SPI_CLK" (at 135.89 97.79 0) (fields_autoplaced)
+  (label "SERVO_SGNL1" (at 135.89 107.95 0) (fields_autoplaced)
     (effects (font (size 1.27 1.27)) (justify left bottom))
   )
-  (label "SERVO_SGNL1" (at 135.89 107.95 0) (fields_autoplaced)
+  (label "SPI_CLK" (at 135.89 100.33 0) (fields_autoplaced)
     (effects (font (size 1.27 1.27)) (justify left bottom))
   )
@@
     (effects (font (size 1.27 1.27)) (justify right bottom))
   )
-  (label "MAG_CS" (at 135.89 118.11 0) (fields_autoplaced)
-    (effects (font (size 1.27 1.27)) (justify left bottom))
-  )
   (label "SPI_MISO" (at 227.33 29.21 180) (fields_autoplaced)
     (effects (font (size 1.27 1.27)) (justify right bottom))
@@
   (label "SD_CLK" (at 227.33 41.91 180) (fields_autoplaced)
     (effects (font (size 1.27 1.27)) (justify right bottom))
+  )
+  (label "MAG_CS" (at 135.89 115.57 0) (fields_autoplaced)
+    (effects (font (size 1.27 1.27)) (justify left bottom))
   )
   (label "SERVO_PWR" (at 210.82 119.38 0) (fields_autoplaced)
@@
     (effects (font (size 1.27 1.27)) (justify right bottom))
   )
-  (label "IMU_CS" (at 135.89 95.25 0) (fields_autoplaced)
-    (effects (font (size 1.27 1.27)) (justify left bottom))
-  )
   (label "RXD" (at 19.05 115.57 180) (fields_autoplaced)
     (effects (font (size 1.27 1.27)) (justify right bottom))
@@
     (effects (font (size 1.27 1.27)) (justify right bottom))
   )
-  (label "SPI_MISO" (at 135.89 115.57 0) (fields_autoplaced)
-    (effects (font (size 1.27 1.27)) (justify left bottom))
-  )
   (label "CAN_TX" (at 15.24 33.02 0) (fields_autoplaced)
     (effects (font (size 1.27 1.27)) (justify left bottom))
   )
-  (label "SPI_MOSI" (at 135.89 100.33 0) (fields_autoplaced)
-    (effects (font (size 1.27 1.27)) (justify left bottom))
-  )

Commit message: final fixes mybe
Parts:
- added TP16: TestPoint, TestPoint:TestPoint_Pad_D1.0mm, symbol Connector:TestPoint
Connections:
- net SERVO_PWR: now also TP16.1
Changed lines of the file:
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@@
   (junction (at 167.64 132.08) (diameter 0) (color 0 0 0 0)
+  )
+  (junction (at 210.82 120.65) (diameter 0) (color 0 0 0 0)
   )
   (junction (at 46.99 135.89) (diameter 0) (color 0 0 0 0)
@@
     (stroke (width 0) (type default))
   )
+  (wire (pts (xy 201.93 120.65) (xy 210.82 120.65))
+    (stroke (width 0) (type default))
+  )
   (wire (pts (xy 234.95 120.65) (xy 234.95 133.35))
     (stroke (width 0) (type default))
@@
         )
       )
+    )
+  )
+  (symbol (lib_id "Connector:TestPoint") (at 201.93 120.65 0) (unit 1)
+    (in_bom yes) (on_board yes) (dnp no)
+    (property "Reference" "TP16" (at 194.31 115.57 0)
+      (effects (font (size 1.27 1.27)) (justify left))
+    )
+    (property "Value" "TestPoint" (at 191.77 118.11 0)
+      (effects (font (size 1.27 1.27)) (justify left))
+    )
+    (property "Footprint" "TestPoint:TestPoint_Pad_D1.0mm" (at 207.01 120.65 0)
+      (effects (font (size 1.27 1.27)) hide)
+    )
+    (property "Datasheet" "~" (at 207.01 120.65 0)
+      (effects (font (size 1.27 1.27)) hide)
+    )
+    (pin "1")
+    (instances
+      (project "Canardboard"
+        (path "/7db990e4-92e1-4f99-b4d2-435bbec1ba83"
+          (reference "TP16") (unit 1)
+        )
+      )
