File: Canardboard.kicad_pcb (KiCad board)
At the start: 4 copper layers, 47 x 60 mm, 173 parts, among them IC1 SIC437DED-T1-GE3, J1 RBUS, J2 USB_C_Receptacle_USB2.0, J3 Micro_SD_Card_Det, J4 Conn_01x02_Male, J5 Conn_01x03_Male, J6 Conn_01x03_Male, J7 Conn_01x03_Male, Q1 PXP012-30QLJ, Q2 PXP012-30QLJ, Q4 PXP012-30QLJ, Q6 PXP012-30QLJ, U1 ESP32-S3, U10 MP28167GQ-A-Z, U2 SN65HVD230, U3 LTC4412xS6, U4 LTC4412xS6, U5 74AHC1G00, U6 74AHC1G08, U9 SC4215, Y1 40MHz±10ppm

Commit message: final fixes mybe
Parts:
- added SERVOPOWER: TestPoint, TestPoint:TestPoint_Pad_D1.0mm, F.Cu at (145.2, 121.5)
- moved C25 6.14 mm to (118.8, 89.5), turned to 90 degrees
- moved R50 4.10 mm to (116.3, 89.0)
- moved C24 4.03 mm to (118.0, 79.0), turned to 0 degrees
- moved U9 3.23 mm to (117.0, 83.8)
- moved C26 3.14 mm to (117.8, 89.5)
- moved R51 1.62 mm to (115.2, 88.0), turned to 180 degrees
Routing:
- net GND: track 60.9 -> 57.6 mm, vias 113 -> 114
- net Net-(U4-CTL): track 29.1 -> 31.0 mm
- net +3.3V: track 49.0 -> 47.6 mm, vias 24 -> 23
- net /rbusmosfets/BatteryPower: track 8.12 -> 7.36 mm
- net RBUS_uC_V: track 74.3 -> 75.0 mm
- net +12V: track 13.1 -> 12.5 mm
- net /rbusmosfets/RBUS_DEPL: track 24.2 -> 23.6 mm
- net /CAN_TX: track 43.9 -> 43.4 mm
- net Net-(Q4-G): track 10.5 -> 10.0 mm
- net /servopower/uC_VOUT: track 3.46 -> 3.02 mm, vias 2 -> 6

Commit message: fixed via bypass capacitors
Parts:
- moved C31 0.60 mm to (113.8, 99.6)
- moved C33 0.60 mm to (112.8, 99.5)
- moved C34 0.60 mm to (114.8, 99.6)
Routing:
- net +3.3V: track 47.6 -> 50.8 mm
- net /SERVOBUCK_EN: track 18.3 -> 19.6 mm

Commit message: final final changes
Parts:
- locked: moved to B.Cu
- moved locked 7.41 mm to (114.8, 92.8), turned to 180 degrees
- renumbered TP6 to MOSI, TP7 to locked
Routing:
- net /SERVOBUCK_EN: track 19.6 -> 16.2 mm
- net +3.3V: track 50.8 -> 52.8 mm
- net /SERVO_SGNL3: track 36.7 -> 38.1 mm
- net /SD_DET: track 29.7 -> 28.9 mm
- net /SPI_CLK: track 12.8 -> 13.5 mm

Commit message: ordering changes
Parts:
- moved J7 1.45 mm to (141.1, 101.2)
- moved J5 1.45 mm to (141.0, 80.3)
- moved J6 1.45 mm to (141.0, 90.8)
Routing:
- net /SERVO_SGNL3: track 38.1 -> 40.2 mm
- net /SERVO_SGNL1: track 33.6 -> 35.6 mm
- net /SERVO_SGNL2: track 17.0 -> 19.0 mm
