File: draft2/Canardboard.kicad_pcb (KiCad board)
At the start: 4 copper layers, 63.6 x 50.8 mm, 106 parts, among them IC1 SIC437DED-T1-GE3, J1 RBUS, J2 USB_C_Receptacle_USB2.0, J3 Micro_SD_Card_Det, J4 Conn_01x02_Male, J5 Conn_01x03_Male, J6 Conn_01x03_Male, J7 Conn_01x03_Male, Q1 SI4143DY-T1-GE3, Q2 SI4143DY-T1-GE3, U1 ESP32-S3, U10 LTC4412xS6, U2 SN65HVD230, U3 LM66200DRLR, U5 MAX77827AEFD+T, U6 SC4215, U8 MMC5983MA, U9 LTC4412xS6, Y1 40MHz±10ppm

Commit message: 31/01/23
Parts:
- added C30: 0.47uF, Capacitor_SMD:C_0603_1608Metric, F.Cu at (152.0, 97.6)
- added C31: 10nF, Capacitor_SMD:C_0603_1608Metric, F.Cu at (151.9, 92.8)
- added C33: 0.1uF, Capacitor_SMD:C_0603_1608Metric, F.Cu at (149.1, 90.2)
- added C34: 2.2uF, Capacitor_SMD:C_0603_1608Metric, F.Cu at (147.1, 97.2)
- added U7: ICM-20608-G, iclr:PQFN50P300X300X80-16N, F.Cu at (143.1, 95.9)
- moved 3V3LED1 9.01 mm to (139.7, 90.1)
- moved C14 7.26 mm to (138.7, 92.1), turned to -90 degrees
- moved C29 5.73 mm to (143.5, 103.6), turned to 180 degrees
- moved Y1 4.97 mm to (136.7, 92.6)
- moved C13 4.27 mm to (137.1, 90.2), turned to 0 degrees
- moved R6 3.27 mm to (141.3, 89.6), turned to 180 degrees
- moved R4 2.57 mm to (141.3, 93.4), turned to 180 degrees
- moved C32 2.14 mm to (147.2, 95.6)
- moved TXLED1 2.06 mm to (141.4, 90.9), turned to 180 degrees
- moved U8 1.97 mm to (143.4, 100.7), turned to -90 degrees
- moved R2 1.66 mm to (141.3, 92.1), turned to 180 degrees
- moved L2 0.10 mm to (135.1, 90.2), turned to 0 degrees
Routing:
- net Net-(J4-Pad1): track 0.00 -> 9.87 mm
- net Net-(C14-Pad1): track 0.00 -> 6.89 mm
- net Net-(C13-Pad1): track 0.00 -> 6.71 mm, vias 0 -> 2
- net GND: track 65.0 -> 70.8 mm
- net Net-(L2-Pad1): track 0.00 -> 4.83 mm
- net +3V3: track 27.7 -> 23.8 mm, vias 1 -> 3
- net Net-(C29-Pad1): track 1.36 -> 0.00 mm

Commit message: 02/02/23
Parts:
- moved JP1 59.0 mm to (122.8, 104.7), turned to 180 degrees
- moved C18 58.2 mm to (118.7, 104.8), turned to -90 degrees
- moved R9 58.1 mm to (118.7, 106.8), turned to 90 degrees
- moved C17 58.0 mm to (120.0, 104.7)
- moved R8 57.7 mm to (115.7, 111.8)
- moved U2 57.3 mm to (119.4, 111.7)
- moved C16 56.9 mm to (119.5, 116.2), turned to 180 degrees
- moved C19 56.7 mm to (122.3, 106.4)
- moved R10 56.1 mm to (120.0, 106.8), turned to -90 degrees
- moved C15 55.2 mm to (119.5, 117.3), turned to 180 degrees
- moved D1 52.9 mm to (115.4, 106.0), turned to 180 degrees
- moved J3 39.3 mm to (144.6, 66.2), turned to 180 degrees
- moved J5 33.9 mm to (159.6, 87.2), turned to -90 degrees
- moved J6 32.6 mm to (159.8, 105.4), turned to -90 degrees
- moved C33 14.7 mm to (147.0, 104.8)
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Routing:
- net GND: track 70.8 -> 88.7 mm, vias 11 -> 13
- net +3V3: track 23.8 -> 38.3 mm, vias 3 -> 6
- net /CAN-: track 0.00 -> 11.2 mm, vias 0 -> 2
- net Net-(R6-Pad2): track 0.00 -> 7.41 mm, vias 0 -> 1
- net /CAN+: track 0.00 -> 6.70 mm
- net Net-(C31-Pad1): track 0.00 -> 5.43 mm
- net Net-(C17-Pad1): track 0.00 -> 4.76 mm
- net /CAN-BUS/Vref: track 2.83 -> 6.13 mm
- net Net-(R8-Pad1): track 0.00 -> 3.24 mm
- net Net-(C30-Pad1): track 0.00 -> 1.50 mm
- net /SERVO_SGNL3: track 0.00 -> 1.25 mm, vias 0 -> 1
- net Net-(C29-Pad1): track 0.00 -> 1.15 mm
- net Net-(3V3LED1-Pad2): track 0.00 -> 1.10 mm
- net /Power/BBOUT: vias 0 -> 2
- net /Power/LX2: vias 7 -> 6
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
Commit message: 04/02/2023
Parts:
- moved TP5 88.2 mm to (134.7, 116.8)
- moved C34 26.0 mm to (121.7, 109.3), turned to 90 degrees
- moved C32 25.2 mm to (133.6, 105.8), turned to 180 degrees
- moved U8 25.1 mm to (133.8, 109.0), turned to 180 degrees
- moved C29 25.0 mm to (133.6, 112.2), turned to 0 degrees
- moved C33 24.1 mm to (123.2, 109.3), turned to 90 degrees
- moved C31 22.3 mm to (124.9, 109.3), turned to 90 degrees
- moved C30 18.4 mm to (126.5, 109.3), turned to 90 degrees
- moved U7 18.2 mm to (129.1, 109.0)
- moved C25 13.5 mm to (121.3, 121.6), turned to 180 degrees
- moved C26 11.8 mm to (123.4, 121.6), turned to 0 degrees
- moved TP7 11.4 mm to (130.2, 122.5), turned to 180 degrees
- moved TP8 10.9 mm to (127.3, 122.5), turned to 180 degrees
- moved J4 10.6 mm to (126.7, 69.5), turned to 90 degrees
- moved R16 10.4 mm to (120.6, 113.3), turned to 180 degrees
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Routing:
- net RBUS_uC_V: track 0.00 -> 37.1 mm, vias 0 -> 2
- net /CAN+: track 6.70 -> 34.7 mm, vias 0 -> 2
- net /CAN-: track 11.2 -> 33.0 mm, vias 2 -> 4
- net GNDA: track 1.96 -> 16.9 mm, vias 0 -> 3
- net +12V: track 62.8 -> 49.5 mm
- net Net-(C44-Pad1): track 5.21 -> 18.2 mm, vias 0 -> 2
- net /BOOT: track 0.00 -> 7.75 mm
- net Net-(J4-Pad1): track 9.87 -> 2.92 mm
- net /SPI_MOSI: track 0.00 -> 6.48 mm
- net /SPI_MISO: track 0.00 -> 5.32 mm
- net Net-(C31-Pad1): track 5.43 -> 10.4 mm
- net /comps/SW: track 0.00 -> 4.74 mm
- net Net-(R8-Pad1): track 3.24 -> 7.98 mm
- net /CHIP_PU: track 10.3 -> 6.28 mm
- net +3V3: track 38.3 -> 40.2 mm, vias 6 -> 5
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Other:
- board size 63.6 x 50.8 mm -> 159.3 x 124.4 mm

Commit message: changes
ch
Routing:
- net GND: vias 14 -> 18
Changed lines of the file:
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@@
   (segment (start 119.97 105.25) (end 119.97 106.13) (width 0.45) (layer "F.Cu") (net 1))
   (segment (start 121.65 108.53) (end 126.44 108.53) (width 0.45) (layer "F.Cu") (net 1))
+  (via (at 104.9 104.2) (size 0.8) (drill 0.4) (layers "F.Cu" "B.Cu") (free) (net 1))
+  (via (at 107.3 104.2) (size 0.8) (drill 0.4) (layers "F.Cu" "B.Cu") (free) (net 1))
   (via (at 128.998508 120.866164) (size 0.6) (drill 0.3) (layers "F.Cu" "B.Cu") (free) (net 1))
   (via (at 122.971 117.45135) (size 0.8) (drill 0.4) (layers "F.Cu" "B.Cu") (net 1))
   (via (at 123.370508 121.945164) (size 0.4) (drill 0.2) (layers "F.Cu" "B.Cu") (net 1))
   (via (at 122.971 118.59135) (size 0.8) (drill 0.4) (layers "F.Cu" "B.Cu") (free) (net 1))
+  (via (at 102.6 104.3) (size 0.8) (drill 0.4) (layers "F.Cu" "B.Cu") (free) (net 1))
   (via (at 127.94 90.53) (size 0.6) (drill 0.3) (layers "F.Cu" "B.Cu") (free) (net 1))
   (via (at 98.9045 97.21) (size 0.8) (drill 0.4) (layers "F.Cu" "B.Cu") (free) (net 1))
   (via (at 97.84 90.55) (size 0.6) (drill 0.3) (layers "F.Cu" "B.Cu") (free) (net 1))
   (via (at 120.011 118.64135) (size 0.8) (drill 0.4) (layers "F.Cu" "B.Cu") (net 1))
+  (via (at 99.8 104.2) (size 0.8) (drill 0.4) (layers "F.Cu" "B.Cu") (free) (net 1))
   (via (at 122.971 117.45135) (size 0.8) (drill 0.4) (layers "F.Cu" "B.Cu") (net 1))
   (via (at 110.87 101) (size 0.6) (drill 0.3) (layers "F.Cu" "B.Cu") (free) (net 1))
@@
   (via (at 119.99 106.13) (size 0.6) (drill 0.3) (layers "F.Cu" "B.Cu") (free) (net 1))
   (via (at 131.660508 119.945164) (size 0.4) (drill 0.2) (layers "F.Cu" "B.Cu") (net 1))
-  (via (at 129.06 93.02) (size 0.6) (drill 0.3) (layers "F.Cu" "B.Cu") (free) (net 1))
+  (via (at 129.06 93.02) (size 0.4) (drill 0.2) (layers "F.Cu" "B.Cu") (free) (net 1))
   (segment (start 131.28 92.05) (end 131.28 93.15) (width 0.45) (layer "F.Cu") (net 2))
   (segment (start 99.83 93.04) (end 100.81 93.04) (width 0.25) (layer "F.Cu") (net 3))
@@
   (segment (start 128.89 94.4625) (end 128.89 93.930025) (width 0.2) (layer "F.Cu") (net 101))
   (segment (start 129.265 93.725) (end 129.45 93.54) (width 0.2) (layer "F.Cu") (net 101))
-  (via (at 129.45 93.54) (size 0.6) (drill 0.3) (layers "F.Cu" "B.Cu") (free) (net 101))
+  (via (at 129.45 93.54) (size 0.4) (drill 0.2) (layers "F.Cu" "B.Cu") (free) (net 101))
   (segment (start 109.21 86.96) (end 108.305 86.96) (width 0.5) (layer "F.Cu") (net 102))
   (segment (start 98.48 87.46) (end 102.04 83.9) (width 0.5) (layer "F.Cu") (net 102))
