File: draft2/comps.kicad_sch (KiCad schematic)
At the start: 33 parts, among them IC1 SIC437DED-T1-GE3, J3 Micro_SD_Card_Det, J4 Conn_01x02_Male, Q1 SI4143DY-T1-GE3, Q2 SI4143DY-T1-GE3, U10 LTC4412xS6, U7 ICM-20608-G, U8 MMC5983MA, U9 LTC4412xS6

Commit message: made everything smaller
:)
Parts:
- C40, C41: footprint iclr:CAPAE830X1050N -> Capacitor_SMD:C_0805_2012Metric
Changed lines of the file:
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@@
       (effects (font (size 1.27 1.27)) (justify left))
     )
-    (property "Footprint" "iclr:CAPAE830X1050N" (id 2) (at 250.19 121.92 0)
+    (property "Footprint" "Capacitor_SMD:C_0805_2012Metric" (id 2) (at 250.19 121.92 0)
       (effects (font (size 1.27 1.27)) hide)
     )
@@
       (effects (font (size 1.27 1.27)) (justify left))
     )
-    (property "Footprint" "iclr:CAPAE830X1050N" (id 2) (at 190.5 123.19 0)
-      (effects (font (size 1.27 1.27)) hide)
-    )
+    (property "Footprint" "Capacitor_SMD:C_0805_2012Metric" (id 2) (at 190.5 123.19 0)
+      (effects (font (size 1.27 1.27)) hide)
+    )

Commit message: changes
ch
Connections:
- net SERVO_PWR: now also L4.1; no longer L4.2
- net SW: now also L4.2; no longer L4.1
Other:
- moved on the sheet: L4
Changed lines of the file:
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@@
     (pin "2")
   )
-  (symbol (lib_id "pspice:INDUCTOR") (at 168.91 55.88 180) (unit 1)
+  (symbol (lib_id "pspice:INDUCTOR") (at 168.91 55.88 0) (unit 1)
     (in_bom yes) (on_board yes) (fields_autoplaced)
-    (property "Reference" "L4" (id 0) (at 168.91 50.8 0))
-    (property "Value" "1.5uH" (id 1) (at 168.91 53.34 0))
+    (property "Reference" "L4" (id 0) (at 168.91 49.53 0))
+    (property "Value" "1.5uH" (id 1) (at 168.91 52.07 0))
     (property "Footprint" "Inductor_SMD:L_1206_3216Metric" (id 2) (at 168.91 55.88 0)
       (effects (font (size 1.27 1.27)) hide)
