File: draft2/Canardboard.kicad_sch (KiCad schematic)
At the start: 48 parts, among them J1 RBUS, U1 ESP32-S3, U5 LTC4411, Y1 40MHz±10ppm

Commit message: used new esp32 board
Parts:
- removed C22: 4.7uF, Capacitor_SMD:C_0603_1608Metric, symbol Device:C_Small
- removed C?: 1uF, Capacitor_SMD:C_0603_1608Metric, symbol Device:C_Small
- removed C?: 10uF, Capacitor_SMD:C_0603_1608Metric, symbol Device:C_Small
- removed C?: 10nF, Capacitor_SMD:C_0603_1608Metric, symbol Device:C_Small
- removed C?: 0.1uF, Capacitor_SMD:C_0603_1608Metric, symbol Device:C_Small
- removed C?: 2.2uF, Capacitor_SMD:C_0603_1608Metric, symbol Device:C_Small
- removed C?: 0.47uF, Capacitor_SMD:C_0603_1608Metric, symbol Device:C_Small
- removed J?: Micro_SD_Card_Det, Connector_Card:microSD_HC_Hirose_DM3AT-SF-PEJM5, symbol Connector:Micro_SD_Card_Det_Hirose_DM3AT
- removed R10: 470, Resistor_SMD:R_0402_1005Metric, symbol Device:R_Small
- removed R?: 10k, symbol Device:R_Small
- removed RXLED1: RX_LED, LED_SMD:LED_0603_1608Metric, symbol Device:LED_Small
- removed U5: LTC4411, Package_TO_SOT_SMD:SOT-23-5, symbol iclr:LTC4411
- removed U?: ICM-20608-G, iclr:PQFN50P300X300X80-16N, symbol iclr:ICM-20608-G
- removed U?: MMC5983MA, iclr:PQFN50P300X300X100-16N, symbol iclr:MMC5983MA
- added R6: 499, Resistor_SMD:R_0402_1005Metric, symbol Device:R_Small
- C1: renamed from C4; footprint (none) -> Capacitor_SMD:C_0402_1005Metric
- C12: value C -> 4.2pF; footprint Capacitor_SMD:C_0603_1608Metric -> Capacitor_SMD:C_0402_1005Metric
- C13, C14: footprint Capacitor_SMD:C_0603_1608Metric -> Capacitor_SMD:C_0402_1005Metric
- L1, L2: footprint (none) -> Inductor_SMD:L_0402_1005Metric
- R5: renamed from R1; value 50 -> 47.5; footprint (none) -> Resistor_SMD:R_0402_1005Metric
- renumbered C1 to C3, C5 to C4, C6 to C5, C7 to C6, C8 to C7, C3 to C8, R7 to R1, R11 to R2, R8 to R3, R14 to R4, R4 to R7
Connections:
- net TXD: now also R6.1
- net RBUS_uC_V: now reaches J1.3 (Pin_3)
- net at U1.49 (U0TXD/PROG/GPIO43): now also R6.2
- no-connect marks 8 -> 3
Other:
- added sheet Power (power.kicad_sch)
- added sheet components (components.kicad_sch)
- moved on the sheet: R2, TXLED1

Commit message: pcb roughly organized
andrei updated his board agaain
Parts:
- added J5, J6, J7: Conn_01x03_Male, Connector_AMASS:AMASS_MR30PW-M_1x03_P3.50mm_Horizontal, symbol Connector:Conn_01x03_Male
Connections:
- net GND: now also J5.1 (Pin_1), J6.1 (Pin_1), J7.1 (Pin_1)
- net SERVO_SGNL1: now reaches U1.36 (SPICLK_N/GPIO48)
- net SERVO_SGNL1: now also J5.3 (Pin_3)
- net SERVO_SGNL2: now reaches U1.37 (SPICLK_P/GPIO47)
- net SERVO_SGNL2: now also J6.3 (Pin_3)
- net SERVO_SGNL3: now reaches U1.44 (MTCK/JTAG/GPIO39)
- net SERVO_SGNL3: now also J7.3 (Pin_3)
- new net SERVO_PWR: J5.2 (Pin_2), J6.2 (Pin_2), J7.2 (Pin_2)
Other:
- removed sheet components
- added sheet comps (comps.kicad_sch)
- note added: "Servo"
