File: Hardware/Canardboard.kicad_pcb (KiCad board)
At the start: 4 copper layers, 47 x 60 mm, 174 parts, among them IC1 SIC437DED-T1-GE3, J1 RBUS, J2 USB_C_Receptacle_USB2.0, J3 Micro_SD_Card_Det, J4 Conn_01x02_Male, J5 Conn_01x03_Male, J6 Conn_01x03_Male, J7 Conn_01x03_Male, Q1 PXP012-30QLJ, Q2 PXP012-30QLJ, Q4 PXP012-30QLJ, Q6 PXP012-30QLJ, U1 ESP32-S3, U10 MP28167GQ-A-Z, U2 SN65HVD230, U3 LTC4412xS6, U4 LTC4412xS6, U5 74AHC1G00, U6 74AHC1G08, U9 SC4215, Y1 40MHz±10ppm

Commit message: Added 3d Models
Parts:
- renumbered locked to 12V, locked to 3V3, locked to BOOT, locked to CLK, locked to CRX, locked to CS, locked to CTX, locked to D+, locked to D-, locked to EN, locked to ICS, locked to IMU, locked to IO, locked to MAG, locked to MCS, locked to MISO, locked to OI, locked to RX, locked to RuCV, locked to S1, locked to S2, locked to S3, locked to SP, locked to TX, locked to TXLED
